File: R_Switch Rev A/R_Switch.sch (KiCad schematic (older format))
At the start: 135 parts, among them J1 Conn_01x04, J2 Conn_01x06, J3 Conn_01x06, J4 Conn_01x05, J5 Conn_01x08, J6 Conn_01x08, Q1 IRF7343PBF, Q2 IRF7343PBF, Q3 IRF7343PBF, Q4 IRF7343PBF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

Commit message: Enable and inhibit inputs
Parts:
- added C5, C6: 0.1, Capacitor_SMD:C_0805_2012Metric_Pad1.15x1.40mm_HandSolder, symbol Device:C_Small
- added D51, D52: D_Small_ALT, Diode_SMD:D_SOD-123, symbol Device:D_Small_ALT
- added J7: Conn_01x03, Connector_Phoenix_MSTB:PhoenixContact_MSTBVA_2,5_3-G-5,08_1x03_P5.08mm_Vertical, symbol Connector_Generic:Conn_01x03
- added Q10, Q9: 2N3906, Package_TO_SOT_THT:TO-92_Inline, symbol Transistor_BJT:2N3906
- added R64, R68, R69, R73, R74, R75: 47K, Resistor_SMD:R_0805_2012Metric_Pad1.15x1.40mm_HandSolder, symbol Device:R_Small
- added R65, R67, R70, R72: 1K0, Resistor_SMD:R_0805_2012Metric_Pad1.15x1.40mm_HandSolder, symbol Device:R_Small
- added R66, R71: 10K, Resistor_SMD:R_0805_2012Metric_Pad1.15x1.40mm_HandSolder, symbol Device:R_Small
Connections:
- wire segments 391 -> 445
Other:
- note added: "DNI"
- note added: "Enable*\nInhibit*\nGND"
- note added: "Optional: Enable and Inhibit Inputs.\n<3v = Active, If not used install R74 and R75 only.\nEnable* must be grounded and Inhibit* must be\n open for unit to work."
- note added: "RB6 Active High Input"
- note added: "RB7 Active High Input"
- note added: "Rev. A Fixed backwards diodes D2, D3.. D11.. \n Added Remote Enable and Disable."
- note removed: "Rev. A Fixed backwards diodes D2, D3.. D11.."
